File: pcb/tt6581.kicad_sch (KiCad schematic)
At the start: 12 parts, among them U1 SN74LVC1G125DBV, U2 OPA1678

Commit message: wip
Parts:
- C1: value C -> 1n
- C2: value C -> 1.1n
- R2: value R -> 5110R
- R3: value R -> 4110R
- R4, R5: value R -> 2870R
Changed lines of the file:
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@@
 			)
 		)
-		(property "Value" "R"
+		(property "Value" "4110R"
 			(at 138.43 80.01 90)
 			(effects
@@
 			)
 		)
-		(property "Value" "R"
+		(property "Value" "5110R"
 			(at 153.67 80.01 90)
 			(effects
@@
 			)
 		)
-		(property "Value" "R"
+		(property "Value" "2870R"
 			(at 137.16 130.81 90)
 			(effects
@@
 			)
 		)
-		(property "Value" "R"
+		(property "Value" "2870R"
 			(at 152.4 130.81 90)
 			(effects
@@
 			)
 		)
-		(property "Value" "C"
+		(property "Value" "1n"
 			(at 165.1 90.1699 0)
 			(effects
@@
 		(dnp no)
 		(property "Reference" "C2"
-			(at 164.338 72.136 90)
-			(effects
-				(font
-					(size 1.27 1.27)
-				)
-			)
-		)
-		(property "Value" "C"
-			(at 157.734 71.628 90)
-			(effects
-				(font
+			(at 164.846 67.818 90)
+			(effects
+				(font
+					(size 1.27 1.27)
+				)
+			)
+		)
+		(property "Value" "1.1n"
+			(at 165.608 71.882 90)
+			(effects
+				(font
